File: KiCAD/keys.kicad_sch (KiCad schematic)
At the start: 204 parts, among them SW1 MX_Lekker, SW10 MX_Lekker, SW11 MX_Lekker, SW12 MX_Lekker, SW13 MX_Lekker, SW14 MX_Lekker, SW15 MX_Lekker, SW16 MX_Lekker, SW17 MX_Lekker, SW18 MX_Lekker, SW19 MX_Lekker, SW2 MX_Lekker, SW20 MX_Lekker, SW21 MX_Lekker, SW22 MX_Lekker, SW23 MX_Lekker, SW24 MX_Lekker, SW25 MX_Lekker, SW26 MX_Lekker, SW27 MX_Lekker, SW28 MX_Lekker, SW29 MX_Lekker, SW3 MX_Lekker, SW30 MX_Lekker, SW31 MX_Lekker, SW32 MX_Lekker, SW33 MX_Lekker, SW34 MX_Lekker, SW35 MX_Lekker, SW36 MX_Lekker, SW37 MX_Lekker, SW38 MX_Lekker, SW39 MX_Lekker, SW4 MX_Lekker, SW40 MX_Lekker, SW41 MX_Lekker, SW42 MX_Lekker, SW43 MX_Lekker, SW44 MX_Lekker, SW45 MX_Lekker, SW46 MX_Lekker, SW47 MX_Lekker, SW48 MX_Lekker, SW49 MX_Lekker, SW5 MX_Lekker, SW50 MX_Lekker, SW51 MX_Lekker, SW52 MX_Lekker, SW53 MX_Lekker, SW54 MX_Lekker, SW55 MX_Lekker, SW56 MX_Lekker, SW57 MX_Lekker, SW58 MX_Lekker, SW59 MX_Lekker, SW6 MX_Lekker, SW60 MX_Lekker, SW61 MX_Lekker, SW62 MX_Lekker, SW63 MX_Lekker, SW64 MX_Lekker, SW65 MX_Lekker, SW66 MX_Lekker, SW67 MX_Lekker, SW68 MX_Lekker, SW7 MX_Lekker, SW8 MX_Lekker, SW9 MX_Lekker, U1 AH49-E, U10 AH49-E, U11 AH49-E, U12 AH49-E, U13 AH49-E, U14 AH49-E, U15 AH49-E, U16 AH49-E, U17 AH49-E, U18 AH49-E, U19 AH49-E, U2 AH49-E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

Commit message: More interim commits
Parts:
- SW1, SW10, SW11, SW12, SW13, SW14, SW15, SW16, SW17, SW18, SW19, SW2, SW20, SW21, SW22, SW23, SW24, SW25, SW26, SW27, SW28, SW29, SW3, SW30, SW31, SW32, SW33, SW34, SW35, SW36, SW37, SW38, SW39, SW4, SW40, SW41, SW42, SW43, SW44, SW45, SW46, SW47, SW48, SW49, SW5, SW50, SW51, SW52, SW53, SW54, SW55, SW56, SW57, SW58, SW59, SW6, SW60, SW61, SW62, SW63, SW64, SW65, SW66, SW67, SW68, SW7, SW8, SW9: footprint (none) -> MX_Only:MX_Lekker

Commit message: Adding more footprints
Parts:
- C1, C10, C11, C12, C13, C14, C15, C16, C17, C18, C19, C2, C20, C21, C22, C23, C24, C25, C26, C27, C28, C29, C3, C30, C31, C32, C33, C34, C35, C36, C37, C38, C39, C4, C40, C41, C42, C43, C44, C45, C46, C47, C48, C49, C5, C50, C51, C52, C53, C54, C55, C56, C57, C58, C59, C6, C60, C61, C62, C63, C64, C65, C66, C67, C68, C7, C8, C9: footprint (none) -> Capacitor_SMD:C_0603_1608Metric_Pad1.08x0.95mm_HandSolder; Part Number (none) -> C0603C104M4RAC7411

Commit message: Update Lekker footprints to include non-1U sizes and stabilizers
Parts:
- SW14: footprint MX_Only:MX_Lekker -> MX_Only:MX_Lekker-2U
- SW16, SW29: footprint MX_Only:MX_Lekker -> MX_Only:MX_Lekker-1.5U
- SW31: footprint MX_Only:MX_Lekker -> MX_Only:MX_Lekker-1.75U
- SW43, SW45: footprint MX_Only:MX_Lekker -> MX_Only:MX_Lekker-2.25U
- SW59, SW60, SW61: footprint MX_Only:MX_Lekker -> MX_Only:MX_Lekker-1.25U
- SW62: footprint MX_Only:MX_Lekker -> MX_Only:MX_Lekker-6.25U-ReversedStabilizers
Changed lines of the file:
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@@
       (effects (font (size 1.27 1.27)) (justify left))
     )
-    (property "Footprint" "MX_Only:MX_Lekker" (id 2) (at 36.83 198.12 0)
+    (property "Footprint" "MX_Only:MX_Lekker-1.25U" (id 2) (at 36.83 198.12 0)
       (effects (font (size 1.27 1.27)) hide)
     )
@@
       (effects (font (size 1.27 1.27)) (justify left))
     )
-    (property "Footprint" "MX_Only:MX_Lekker" (id 2) (at 350.52 76.2 0)
+    (property "Footprint" "MX_Only:MX_Lekker-1.5U" (id 2) (at 350.52 76.2 0)
       (effects (font (size 1.27 1.27)) hide)
     )
@@
       (effects (font (size 1.27 1.27)) (justify left))
     )
-    (property "Footprint" "MX_Only:MX_Lekker" (id 2) (at 36.83 116.84 0)
+    (property "Footprint" "MX_Only:MX_Lekker-1.75U" (id 2) (at 36.83 116.84 0)
       (effects (font (size 1.27 1.27)) hide)
     )
@@
       (effects (font (size 1.27 1.27)) (justify left))
     )
-    (property "Footprint" "MX_Only:MX_Lekker" (id 2) (at 85.09 198.12 0)
+    (property "Footprint" "MX_Only:MX_Lekker-1.25U" (id 2) (at 85.09 198.12 0)
       (effects (font (size 1.27 1.27)) hide)
     )
@@
       (effects (font (size 1.27 1.27)) (justify left))
     )
-    (property "Footprint" "MX_Only:MX_Lekker" (id 2) (at 36.83 76.2 0)
+    (property "Footprint" "MX_Only:MX_Lekker-1.5U" (id 2) (at 36.83 76.2 0)
       (effects (font (size 1.27 1.27)) hide)
     )
@@
       (effects (font (size 1.27 1.27)) (justify left))
     )
-    (property "Footprint" "MX_Only:MX_Lekker" (id 2) (at 36.83 157.48 0)
+    (property "Footprint" "MX_Only:MX_Lekker-2.25U" (id 2) (at 36.83 157.48 0)
       (effects (font (size 1.27 1.27)) hide)
     )
@@
       (effects (font (size 1.27 1.27)) (justify left))
     )
-    (property "Footprint" "MX_Only:MX_Lekker" (id 2) (at 350.52 35.56 0)
+    (property "Footprint" "MX_Only:MX_Lekker-2U" (id 2) (at 350.52 35.56 0)
       (effects (font (size 1.27 1.27)) hide)
     )
@@
       (effects (font (size 1.27 1.27)) (justify left))
     )
-    (property "Footprint" "MX_Only:MX_Lekker" (id 2) (at 60.96 198.12 0)
+    (property "Footprint" "MX_Only:MX_Lekker-1.25U" (id 2) (at 60.96 198.12 0)
       (effects (font (size 1.27 1.27)) hide)
     )
@@
       (effects (font (size 1.27 1.27)) (justify left))
     )
-    (property "Footprint" "MX_Only:MX_Lekker" (id 2) (at 326.39 116.84 0)
+    (property "Footprint" "MX_Only:MX_Lekker-2.25U" (id 2) (at 326.39 116.84 0)
       (effects (font (size 1.27 1.27)) hide)
     )
@@
       (effects (font (size 1.27 1.27)) (justify left))
     )
-    (property "Footprint" "MX_Only:MX_Lekker" (id 2) (at 181.61 198.12 0)
+    (property "Footprint" "MX_Only:MX_Lekker-6.25U-ReversedStabilizers" (id 2) (at 181.61 198.12 0)
       (effects (font (size 1.27 1.27)) hide)
     )

Commit message: Fix right shift not having the 1.75U footprint
Parts:
- SW56: footprint MX_Only:MX_Lekker -> MX_Only:MX_Lekker-1.75U
Changed lines of the file:
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@@
       (effects (font (size 1.27 1.27)) (justify left))
     )
-    (property "Footprint" "MX_Only:MX_Lekker" (id 2) (at 326.39 157.48 0)
+    (property "Footprint" "MX_Only:MX_Lekker-1.75U" (id 2) (at 326.39 157.48 0)
       (effects (font (size 1.27 1.27)) hide)
     )

Commit message: pushing various updates
Parts:
- U1, U10, U11, U12, U13, U14, U15, U16, U17, U18, U19, U2, U20, U21, U22, U23, U24, U25, U26, U27, U28, U29, U3, U30, U31, U32, U33, U34, U35, U36, U37, U38, U39, U4, U40, U41, U42, U43, U44, U45, U46, U47, U48, U49, U5, U50, U51, U52, U53, U54, U55, U56, U57, U58, U59, U6, U60, U61, U62, U63, U64, U65, U66, U67, U68, U7, U8, U9: value AH49-E -> DRV5055Z3QDBZT; Part Number (none) -> DRV5055Z3QDBZT
