File: KiCAD/led_drivers.kicad_sch (KiCad schematic)
At the start: 25 parts, among them IC5 IS31FL3733B-TQLS4, IC6 IS31FL3733B-TQLS4

Commit message: Adding more footprints
Parts:
- C71, C74, C76, C78, C80, C82: Part Number (none) -> C0603C104M4RAC7411
Changed lines of the file:
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@@
+      (effects (font (size 1.27 1.27)) hide)
+    )
+    (property "Part Number" "C0603C104M4RAC7411" (id 4) (at 121.92 124.46 0)
       (effects (font (size 1.27 1.27)) hide)
     )
@@
     )
     (property "Datasheet" "~" (id 3) (at 138.43 60.96 0)
+      (effects (font (size 1.27 1.27)) hide)
+    )
+    (property "Part Number" "C0603C104M4RAC7411" (id 4) (at 138.43 60.96 0)
       (effects (font (size 1.27 1.27)) hide)
     )
@@
     )
     (property "Datasheet" "~" (id 3) (at 250.19 119.38 0)
+      (effects (font (size 1.27 1.27)) hide)
+    )
+    (property "Part Number" "C0603C104M4RAC7411" (id 4) (at 250.19 119.38 0)
       (effects (font (size 1.27 1.27)) hide)
     )
@@
       (effects (font (size 1.27 1.27)) hide)
     )
+    (property "Part Number" "C0603C104M4RAC7411" (id 4) (at 63.5 137.16 0)
+      (effects (font (size 1.27 1.27)) hide)
+    )
     (pin "1")
     (pin "2")
@@
       (effects (font (size 1.27 1.27)) hide)
     )
+    (property "Part Number" "C0603C104M4RAC7411" (id 4) (at 256.54 50.8 0)
+      (effects (font (size 1.27 1.27)) hide)
+    )
     (pin "1")
     (pin "2")
@@
       (effects (font (size 1.27 1.27)) hide)
     )
+    (property "Part Number" "C0603C104M4RAC7411" (id 4) (at 232.41 135.89 0)
+      (effects (font (size 1.27 1.27)) hide)
+    )

Commit message: Finished initial routing of PCB
Parts:
- added TP6: TestPoint, TestPoint:TestPoint_Pad_D1.0mm, symbol Connector:TestPoint
Connections:
- net SHUTDOWN_JP: no longer names the net of IC5.46 (SDB), R3.2, TP1.1
- net SHUTDOWN_JP: no longer IC6.46 (SDB), R4.2
- new net: IC6.46 (SDB), R4.2, TP6.1
Changed lines of the file:
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@@
-    (stroke (width 0) (type default) (color 0 0 0 0))
-  )
-  (wire (pts (xy 152.4 26.67) (xy 158.75 26.67))
     (stroke (width 0) (type default) (color 0 0 0 0))
   )
@@
     )
   )
-  (global_label "SHUTDOWN_JP" (shape input) (at 185.42 48.26 180) (fields_autoplaced)
-    (effects (font (size 1.27 1.27)) (justify right))
-    (property "Intersheet References" "${INTERSHEET_REFS}" (id 0) (at 169.5812 48.1806 0)
-      (effects (font (size 1.27 1.27)) (justify right) hide)
-    )
-  )
   (global_label "LED1_Col9" (shape input) (at 110.49 107.95 0) (fields_autoplaced)
     (effects (font (size 1.27 1.27)) (justify left))
@@
     )
   )
-  (global_label "SHUTDOWN_JP" (shape input) (at 69.85 46.99 180) (fields_autoplaced)
-    (effects (font (size 1.27 1.27)) (justify right))
-    (property "Intersheet References" "${INTERSHEET_REFS}" (id 0) (at 54.0112 46.9106 0)
-      (effects (font (size 1.27 1.27)) (justify right) hide)
-    )
-  )
   (global_label "LED_Row_R3" (shape input) (at 168.91 95.25 180) (fields_autoplaced)
     (effects (font (size 1.27 1.27)) (justify right))
@@
     (property "Intersheet References" "${INTERSHEET_REFS}" (id 0) (at 79.9306 145.6812 90)
       (effects (font (size 1.27 1.27)) (justify left) hide)
-    )
-  )
-  (global_label "SHUTDOWN_JP" (shape input) (at 152.4 26.67 180) (fields_autoplaced)
-    (effects (font (size 1.27 1.27)) (justify right))
-    (property "Intersheet References" "${INTERSHEET_REFS}" (id 0) (at 136.5612 26.5906 0)
-      (effects (font (size 1.27 1.27)) (justify right) hide)
     )
   )
@@
     (pin "1")
     (pin "2")
-  )
-  (symbol (lib_id "Connector:TestPoint") (at 158.75 26.67 270) (unit 1)
-    (in_bom yes) (on_board yes) (fields_autoplaced)
-    (property "Reference" "TP1" (id 0) (at 163.83 25.3999 90)
-      (effects (font (size 1.27 1.27)) (justify left))
-    )
-    (property "Value" "TestPoint" (id 1) (at 163.83 27.9399 90)
-      (effects (font (size 1.27 1.27)) (justify left))
-    )
-    (property "Footprint" "TestPoint:TestPoint_Pad_D1.0mm" (id 2) (at 158.75 31.75 0)
-      (effects (font (size 1.27 1.27)) hide)
-    )
-    (property "Datasheet" "~" (id 3) (at 158.75 31.75 0)
-      (effects (font (size 1.27 1.27)) hide)
-    )
-    (pin "1")
   )
   (symbol (lib_id "power:GND") (at 118.11 85.09 90) (unit 1)
@@
     (pin "1")
   )
+  (symbol (lib_id "Connector:TestPoint") (at 185.42 48.26 90) (unit 1)
+    (in_bom yes) (on_board yes) (fields_autoplaced)
+    (property "Reference" "TP6" (id 0) (at 182.118 41.91 90))
+    (property "Value" "TestPoint" (id 1) (at 182.118 44.45 90))
+    (property "Footprint" "TestPoint:TestPoint_Pad_D1.0mm" (id 2) (at 185.42 43.18 0)
+      (effects (font (size 1.27 1.27)) hide)
+    )
+    (property "Datasheet" "~" (id 3) (at 185.42 43.18 0)
+      (effects (font (size 1.27 1.27)) hide)
+    )
+    (pin "1")
+  )
   (symbol (lib_id "Device:R_US") (at 177.8 58.42 90) (unit 1)
     (in_bom yes) (on_board yes)
@@
       (effects (font (size 1.27 1.27)) hide)
     )
+    (pin "1")
+  )
+  (symbol (lib_id "Connector:TestPoint") (at 69.85 46.99 90) (unit 1)
+    (in_bom yes) (on_board yes) (fields_autoplaced)
+    (property "Reference" "TP1" (id 0) (at 66.548 40.64 90))
+    (property "Value" "TestPoint" (id 1) (at 66.548 43.18 90))
+    (property "Footprint" "TestPoint:TestPoint_Pad_D1.0mm" (id 2) (at 69.85 41.91 0)
+      (effects (font (size 1.27 1.27)) hide)
+    )
+    (property "Datasheet" "~" (id 3) (at 69.85 41.91 0)
+      (effects (font (size 1.27 1.27)) hide)
+    )

Commit message: pushing various updates
Parts:
- C69, C70, C72, C73, C75, C77, C79, C81: Part Number (none) -> C1608X7R1C474K080AC
- R1, R2: Part Number (none) -> RMCF0603FT4K70
- R3, R4, R5, R6: Part Number (none) -> RMCF0603FT100K
- R7, R8: Part Number (none) -> ERJ-3EKF2002V
Changed lines of the file:
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@@
+      (effects (font (size 1.27 1.27)) hide)
+    )
+    (property "Part Number" "C1608X7R1C474K080AC" (id 4) (at 100.33 52.07 0)
       (effects (font (size 1.27 1.27)) hide)
     )
@@
       (effects (font (size 1.27 1.27)) hide)
     )
+    (property "Part Number" "ERJ-3EKF2002V" (id 4) (at 110.49 85.09 0)
+      (effects (font (size 1.27 1.27)) hide)
+    )
     (pin "1")
     (pin "2")
@@
     )
     (property "Datasheet" "~" (id 3) (at 50.8 137.16 0)
+      (effects (font (size 1.27 1.27)) hide)
+    )
+    (property "Part Number" "C1608X7R1C474K080AC" (id 4) (at 50.8 137.16 0)
       (effects (font (size 1.27 1.27)) hide)
     )
@@
       (effects (font (size 1.27 1.27)) hide)
     )
+    (property "Part Number" "RMCF0603FT100K" (id 4) (at 67.31 52.07 0)
+      (effects (font (size 1.27 1.27)) hide)
+    )
     (pin "1")
     (pin "2")
@@
       (effects (font (size 1.27 1.27)) hide)
     )
+    (property "Part Number" "C1608X7R1C474K080AC" (id 4) (at 219.71 135.89 0)
+      (effects (font (size 1.27 1.27)) hide)
+    )
     (pin "1")
     (pin "2")
@@
     )
     (property "Datasheet" "~" (id 3) (at 125.73 60.96 0)
+      (effects (font (size 1.27 1.27)) hide)
+    )
+    (property "Part Number" "C1608X7R1C474K080AC" (id 4) (at 125.73 60.96 0)
       (effects (font (size 1.27 1.27)) hide)
     )
@@
       (effects (font (size 1.27 1.27)) hide)
     )
+    (property "Part Number" "ERJ-3EKF2002V" (id 4) (at 229.87 85.09 0)
+      (effects (font (size 1.27 1.27)) hide)
+    )
     (pin "1")
     (pin "2")
@@
       (effects (font (size 1.27 1.27)) hide)
     )
+    (property "Part Number" "C1608X7R1C474K080AC" (id 4) (at 109.22 124.46 0)
+      (effects (font (size 1.27 1.27)) hide)
+    )
     (pin "1")
     (pin "2")
@@
     )
     (property "Datasheet" "~" (id 3) (at 237.49 119.38 0)
+      (effects (font (size 1.27 1.27)) hide)
+    )
+    (property "Part Number" "C1608X7R1C474K080AC" (id 4) (at 237.49 119.38 0)
       (effects (font (size 1.27 1.27)) hide)
     )
@@
       (effects (font (size 1.27 1.27)) hide)
     )
+    (property "Part Number" "RMCF0603FT4K70" (id 4) (at 99.06 31.75 0)
+      (effects (font (size 1.27 1.27)) hide)
+    )
     (pin "1")
     (pin "2")
@@
       (effects (font (size 1.27 1.27)) hide)
     )
+    (property "Part Number" "RMCF0603FT100K" (id 4) (at 62.23 57.15 0)
+      (effects (font (size 1.27 1.27)) hide)
+    )
     (pin "1")
     (pin "2")
@@
       (effects (font (size 1.27 1.27)) hide)
     )
+    (property "Part Number" "RMCF0603FT100K" (id 4) (at 185.42 53.34 0)
+      (effects (font (size 1.27 1.27)) hide)
+    )
     (pin "1")
     (pin "2")
@@
     )
     (property "Datasheet" "~" (id 3) (at 243.84 50.8 0)
+      (effects (font (size 1.27 1.27)) hide)
+    )
+    (property "Part Number" "C1608X7R1C474K080AC" (id 4) (at 243.84 50.8 0)
       (effects (font (size 1.27 1.27)) hide)
     )
@@
       (effects (font (size 1.27 1.27)) hide)
     )
+    (property "Part Number" "RMCF0603FT100K" (id 4) (at 177.8 58.42 0)
+      (effects (font (size 1.27 1.27)) hide)
+    )
     (pin "1")
     (pin "2")
@@
       (effects (font (size 1.27 1.27)) hide)
     )
+    (property "Part Number" "C1608X7R1C474K080AC" (id 4) (at 217.17 40.64 0)
+      (effects (font (size 1.27 1.27)) hide)
+    )
     (pin "1")
     (pin "2")
@@
       (effects (font (size 1.27 1.27)) hide)
     )
+    (property "Part Number" "RMCF0603FT4K70" (id 4) (at 106.68 31.75 0)
+      (effects (font (size 1.27 1.27)) hide)
+    )
