File: KiCAD/led_matrix.kicad_sch (KiCad schematic)
At the start: 67 parts

Commit message: More script and schematic updates
Parts:
- added S15: QBLP677R-RGB, random-keyboard-parts:QBLP677R-RGB-square_cutout, symbol Device:LED_BGRA
- renumbered S15 to S16, S16 to S17, S17 to S18, S18 to S19, S19 to S20, S20 to S21, S21 to S22, S22 to S23, S23 to S24, S24 to S25, S25 to S26, S26 to S27, S27 to S28, S28 to S29, S29 to S30, S30 to S31, S31 to S32, S32 to S33, S33 to S34, S34 to S35, S35 to S36, S36 to S37, S37 to S38, S38 to S39, S39 to S40, S40 to S41, S41 to S42, S42 to S43, S43 to S44, S44 to S45, S45 to S46, S46 to S47, S47 to S48, S48 to S49, S49 to S50, S50 to S51, S51 to S52, S52 to S53, S53 to S54, S54 to S55, S55 to S56, S56 to S57, S57 to S58, S58 to S59, S59 to S60, S60 to S61, S61 to S62, S62 to S63, S63 to S64, S64 to S65, S65 to S66, S66 to S67, S67 to S68
Connections:
- net LED1_Col14: now also S15.4 (A)
- net LED_Row_B0: now also S15.1 (BK)
- net LED_Row_G0: now also S15.2 (GK)
- net LED_Row_R0: now also S15.3 (RK)

Commit message: pushing various updates
Parts:
- S1, S10, S11, S12, S13, S14, S15, S16, S17, S18, S19, S2, S20, S21, S22, S23, S24, S25, S26, S27, S28, S29, S3, S30, S31, S32, S33, S34, S35, S36, S37, S38, S39, S4, S40, S41, S42, S43, S44, S45, S46, S47, S48, S49, S5, S50, S51, S52, S53, S54, S55, S56, S57, S58, S59, S6, S60, S61, S62, S63, S64, S65, S66, S67, S68, S7, S8, S9: Part Number (none) -> QBLP677R-RGB
