File: KiCAD/misc.kicad_sch (KiCad schematic)
At the start: 12 parts

Commit message: More interim commits
Parts:
- gave numbers to parts that had none: 12
Changed lines of the file:
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@@
   (symbol (lib_id "Device:R_US") (at 167.64 58.42 90) (unit 1)
     (in_bom yes) (on_board yes) (fields_autoplaced)
-    (property "Reference" "R?" (id 0) (at 167.64 52.07 90))
+    (property "Reference" "R24" (id 0) (at 167.64 52.07 90))
     (property "Value" "27" (id 1) (at 167.64 54.61 90))
     (property "Footprint" "Resistor_SMD:R_0603_1608Metric_Pad0.98x0.95mm_HandSolder" (id 2) (at 167.894 57.404 90)
@@
   (symbol (lib_id "power:PWR_FLAG") (at 157.48 64.77 270) (unit 1)
     (in_bom yes) (on_board yes)
-    (property "Reference" "#FLG?" (id 0) (at 159.385 64.77 0)
+    (property "Reference" "#FLG02" (id 0) (at 159.385 64.77 0)
       (effects (font (size 1.27 1.27)) hide)
     )
@@
   (symbol (lib_id "power:+5V") (at 157.48 52.07 0) (unit 1)
     (in_bom yes) (on_board yes) (fields_autoplaced)
-    (property "Reference" "#PWR?" (id 0) (at 157.48 55.88 0)
+    (property "Reference" "#PWR0266" (id 0) (at 157.48 55.88 0)
       (effects (font (size 1.27 1.27)) hide)
     )
@@
   (symbol (lib_id "Connector:TestPoint") (at 54.61 44.45 90) (unit 1)
     (in_bom yes) (on_board yes)
-    (property "Reference" "TP?" (id 0) (at 48.26 44.45 90))
+    (property "Reference" "TP2" (id 0) (at 48.26 44.45 90))
     (property "Value" "TestPoint" (id 1) (at 44.45 45.72 90)
       (effects (font (size 1.27 1.27)) hide)
@@
   (symbol (lib_id "Regulator_Linear:NCP1117-3.3_SOT223") (at 73.66 50.8 0) (unit 1)
     (in_bom yes) (on_board yes) (fields_autoplaced)
-    (property "Reference" "U?" (id 0) (at 73.66 43.18 0))
+    (property "Reference" "U72" (id 0) (at 73.66 43.18 0))
     (property "Value" "NCP1117-3.3_SOT223" (id 1) (at 73.66 45.72 0))
     (property "Footprint" "Package_TO_SOT_SMD:SOT-223-3_TabPin2" (id 2) (at 73.66 45.72 0)
@@
   (symbol (lib_id "power:+3.3V") (at 71.12 128.27 0) (unit 1)
     (in_bom yes) (on_board yes)
-    (property "Reference" "#PWR?" (id 0) (at 71.12 132.08 0)
+    (property "Reference" "#PWR0271" (id 0) (at 71.12 132.08 0)
       (effects (font (size 1.27 1.27)) hide)
     )
@@
   (symbol (lib_id "Connector:TestPoint") (at 92.71 104.14 90) (unit 1)
     (in_bom yes) (on_board yes)
-    (property "Reference" "TP?" (id 0) (at 87.63 104.14 90)
+    (property "Reference" "TP5" (id 0) (at 87.63 104.14 90)
       (effects (font (size 1.27 1.27)) (justify left))
     )
@@
   (symbol (lib_id "power:+5V") (at 55.88 43.18 0) (unit 1)
     (in_bom yes) (on_board yes) (fields_autoplaced)
-    (property "Reference" "#PWR?" (id 0) (at 55.88 46.99 0)
+    (property "Reference" "#PWR0263" (id 0) (at 55.88 46.99 0)
       (effects (font (size 1.27 1.27)) hide)
     )
@@
   (symbol (lib_id "power:+3.3VA") (at 88.9 43.18 0) (unit 1)
     (in_bom yes) (on_board yes) (fields_autoplaced)
-    (property "Reference" "#PWR?" (id 0) (at 88.9 46.99 0)
+    (property "Reference" "#PWR0264" (id 0) (at 88.9 46.99 0)
       (effects (font (size 1.27 1.27)) hide)
     )
@@
   (symbol (lib_id "power:+3.3V") (at 86.36 128.27 0) (unit 1)
     (in_bom yes) (on_board yes) (fields_autoplaced)
-    (property "Reference" "#PWR?" (id 0) (at 86.36 132.08 0)
+    (property "Reference" "#PWR0272" (id 0) (at 86.36 132.08 0)
       (effects (font (size 1.27 1.27)) hide)
     )
@@
   (symbol (lib_id "power:GND") (at 55.88 62.23 0) (unit 1)
     (in_bom yes) (on_board yes) (fields_autoplaced)
-    (property "Reference" "#PWR?" (id 0) (at 55.88 68.58 0)
+    (property "Reference" "#PWR0268" (id 0) (at 55.88 68.58 0)
       (effects (font (size 1.27 1.27)) hide)
     )
@@
   (symbol (lib_id "Device:C") (at 55.88 54.61 180) (unit 1)
     (in_bom yes) (on_board yes)
-    (property "Reference" "C?" (id 0) (at 50.8 53.34 0)
+    (property "Reference" "C98" (id 0) (at 50.8 53.34 0)
       (effects (font (size 1.27 1.27)) (justify right))
     )
@@
   (symbol (lib_id "power:PWR_FLAG") (at 157.48 53.34 270) (unit 1)
     (in_bom yes) (on_board yes) (fields_autoplaced)
-    (property "Reference" "#FLG?" (id 0) (at 159.385 53.34 0)
+    (property "Reference" "#FLG01" (id 0) (at 159.385 53.34 0)
       (effects (font (size 1.27 1.27)) hide)
     )
@@
   (symbol (lib_id "Device:R_US") (at 71.12 133.35 0) (unit 1)
     (in_bom yes) (on_board yes)
-    (property "Reference" "R?" (id 0) (at 74.93 132.08 0))
+    (property "Reference" "R26" (id 0) (at 74.93 132.08 0))
     (property "Value" "DNI" (id 1) (at 74.93 134.62 0))
     (property "Footprint" "Resistor_SMD:R_0603_1608Metric_Pad0.98x0.95mm_HandSolder" (id 2) (at 72.136 133.604 90)
@@
   (symbol (lib_id "Connector:TestPoint") (at 92.71 99.06 90) (unit 1)
     (in_bom yes) (on_board yes)
-    (property "Reference" "TP?" (id 0) (at 87.63 99.06 90)
+    (property "Reference" "TP3" (id 0) (at 87.63 99.06 90)
       (effects (font (size 1.27 1.27)) (justify left))
     )
@@
   (symbol (lib_id "Connector:TestPoint") (at 92.71 101.6 90) (unit 1)
     (in_bom yes) (on_board yes)
-    (property "Reference" "TP?" (id 0) (at 87.63 101.6 90)
+    (property "Reference" "TP4" (id 0) (at 87.63 101.6 90)
       (effects (font (size 1.27 1.27)) (justify left))
     )
@@
   (symbol (lib_id "Connector_Generic:Conn_01x04") (at 149.86 58.42 0) (mirror y) (unit 1)
     (in_bom yes) (on_board yes) (fields_autoplaced)
-    (property "Reference" "J?" (id 0) (at 149.86 49.53 0))
+    (property "Reference" "J1" (id 0) (at 149.86 49.53 0))
     (property "Value" "Conn_01x04" (id 1) (at 149.86 52.07 0))
     (property "Footprint" "Connector_JST:JST_SH_SM04B-SRSS-TB_1x04-1MP_P1.00mm_Horizontal" (id 2) (at 149.86 58.42 0)
@@
   (symbol (lib_id "Device:R_US") (at 167.64 60.96 270) (unit 1)
     (in_bom yes) (on_board yes)
-    (property "Reference" "R?" (id 0) (at 167.64 63.5 90))
+    (property "Reference" "R25" (id 0) (at 167.64 63.5 90))
     (property "Value" "27" (id 1) (at 167.64 66.04 90))
     (property "Footprint" "Resistor_SMD:R_0603_1608Metric_Pad0.98x0.95mm_HandSolder" (id 2) (at 167.386 61.976 90)
@@
   (symbol (lib_id "power:GNDPWR") (at 60.96 60.96 0) (unit 1)
     (in_bom yes) (on_board yes) (fields_autoplaced)
-    (property "Reference" "#PWR?" (id 0) (at 60.96 66.04 0)
+    (property "Reference" "#PWR0267" (id 0) (at 60.96 66.04 0)
       (effects (font (size 1.27 1.27)) hide)
     )
@@
   (symbol (lib_id "power:GND") (at 157.48 66.04 0) (unit 1)
     (in_bom yes) (on_board yes) (fields_autoplaced)
-    (property "Reference" "#PWR?" (id 0) (at 157.48 72.39 0)
+    (property "Reference" "#PWR0269" (id 0) (at 157.48 72.39 0)
       (effects (font (size 1.27 1.27)) hide)
     )
@@
   (symbol (lib_id "Connector_Generic:Conn_01x03") (at 46.99 140.97 0) (mirror y) (unit 1)
     (in_bom yes) (on_board yes) (fields_autoplaced)
-    (property "Reference" "J?" (id 0) (at 46.99 132.08 0))
+    (property "Reference" "J2" (id 0) (at 46.99 132.08 0))
     (property "Value" "Conn_01x03" (id 1) (at 46.99 134.62 0))
     (property "Footprint" "Connector_PinHeader_2.54mm:PinHeader_1x03_P2.54mm_Vertical" (id 2) (at 46.99 140.97 0)
@@
   (symbol (lib_id "power:GND") (at 54.61 146.05 0) (unit 1)
     (in_bom yes) (on_board yes) (fields_autoplaced)
-    (property "Reference" "#PWR?" (id 0) (at 54.61 152.4 0)
+    (property "Reference" "#PWR0273" (id 0) (at 54.61 152.4 0)
       (effects (font (size 1.27 1.27)) hide)
     )
@@
   (symbol (lib_id "Device:R_US") (at 86.36 133.35 0) (unit 1)
     (in_bom yes) (on_board yes)
-    (property "Reference" "R?" (id 0) (at 90.17 132.08 0))
+    (property "Reference" "R27" (id 0) (at 90.17 132.08 0))
     (property "Value" "DNI" (id 1) (at 90.17 134.62 0))
     (property "Footprint" "Resistor_SMD:R_0603_1608Metric_Pad0.98x0.95mm_HandSolder" (id 2) (at 87.376 133.604 90)
@@
   (symbol (lib_id "power:+3.3V") (at 96.52 43.18 0) (unit 1)
     (in_bom yes) (on_board yes) (fields_autoplaced)
-    (property "Reference" "#PWR?" (id 0) (at 96.52 46.99 0)
+    (property "Reference" "#PWR0265" (id 0) (at 96.52 46.99 0)
       (effects (font (size 1.27 1.27)) hide)
     )
@@
   (symbol (lib_id "power:GND") (at 95.25 107.95 0) (unit 1)
     (in_bom yes) (on_board yes) (fields_autoplaced)
-    (property "Reference" "#PWR?" (id 0) (at 95.25 114.3 0)
-      (effects (font (size 1.27 1.27)) hide)
-    )
+    (property "Reference" "#PWR0270" (id 0) (at 95.25 114.3 0)
+      (effects (font (size 1.27 1.27)) hide)
+    )

Commit message: Finished initial routing of PCB
Changed lines of the file:
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@@
-    (stroke (width 0) (type default) (color 0 0 0 0))
-  )
-  (wire (pts (xy 88.9 50.8) (xy 88.9 43.18))
     (stroke (width 0) (type default) (color 0 0 0 0))
   )
@@
     (stroke (width 0) (type default) (color 0 0 0 0))
   )
+  (wire (pts (xy 88.9 43.18) (xy 88.9 50.8))
+    (stroke (width 0) (type default) (color 0 0 0 0))
+  )

Commit message: pushing various updates
Parts:
- J1: Part Number (none) -> SM04B-SRSS-TB
- R24, R25: Part Number (none) -> RC0603FR-1327RL
Changed lines of the file:
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@@
+      (effects (font (size 1.27 1.27)) hide)
+    )
+    (property "Part Number" "RC0603FR-1327RL" (id 4) (at 167.64 58.42 0)
       (effects (font (size 1.27 1.27)) hide)
     )
@@
       (effects (font (size 1.27 1.27)) hide)
     )
+    (property "Part Number" "SM04B-SRSS-TB" (id 4) (at 149.86 58.42 0)
+      (effects (font (size 1.27 1.27)) hide)
+    )
     (pin "1")
     (pin "2")
@@
       (effects (font (size 1.27 1.27)) hide)
     )
+    (property "Part Number" "RC0603FR-1327RL" (id 4) (at 167.64 60.96 0)
+      (effects (font (size 1.27 1.27)) hide)
+    )
